File: sch/main.brd (EAGLE design)
At the start: 49.2 x 49.5 mm, 20 parts, among them X1 1503_02

Commit message: [ update ] schematics
Routing:
- net N$1: track 45.4 -> 42.2 mm
Other:
- board text added: "texane@gmail.com"
- board text added: "v0000"
Changed lines of the file:
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@@
 <wire x1="49.2" y1="49.52" x2="0" y2="49.52" width="0" layer="20"/>
 <wire x1="0" y1="49.52" x2="0" y2="0" width="0" layer="20"/>
+<text x="2.54" y="45.72" size="0.8128" layer="25">texane@gmail.com</text>
+<text x="2.54" y="46.99" size="0.8128" layer="25">v0000</text>
 </plain>
 <attributes>
@@
 <wire x1="13.97" y1="46.36" x2="13.97" y2="43.18" width="0.8128" layer="1"/>
 <wire x1="13.97" y1="43.18" x2="25.4" y2="43.18" width="0.8128" layer="1"/>
-<wire x1="25.4" y1="43.18" x2="25.4" y2="43.31" width="0.8128" layer="1"/>
-<wire x1="25.4" y1="43.31" x2="34.8488" y2="43.31" width="0.8128" layer="1"/>
-<wire x1="34.8488" y1="43.31" x2="34.8488" y2="41.91" width="0.8128" layer="1"/>
 <wire x1="38.1" y1="34.16" x2="31.75" y2="34.16" width="0.8128" layer="1"/>
 <wire x1="31.75" y1="34.16" x2="29.21" y2="34.16" width="0.8128" layer="1"/>
 <wire x1="34.8488" y1="41.91" x2="31.75" y2="41.91" width="0.8128" layer="1"/>
 <wire x1="31.75" y1="41.91" x2="31.75" y2="34.16" width="0.8128" layer="1"/>
+<wire x1="31.75" y1="41.91" x2="31.75" y2="43.18" width="0.8128" layer="1"/>
+<wire x1="31.75" y1="43.18" x2="25.4" y2="43.18" width="0.8128" layer="1"/>
+<wire x1="25.4" y1="43.18" x2="25.4" y2="43.31" width="0.8128" layer="1"/>
 </signal>
 <signal name="VDD_ADC">
@@
 <contactref element="R5" pad="1"/>
 <contactref element="X1" pad="3"/>
-<wire x1="21.53" y1="37.51" x2="25.4" y2="37.51" width="0.8128" layer="1"/>
-<wire x1="25.4" y1="37.51" x2="25.4" y2="36.96" width="0.8128" layer="1"/>
 <wire x1="25.4" y1="36.96" x2="25.4" y2="40.51" width="0.8128" layer="1"/>
+<wire x1="25.4" y1="36.96" x2="21.53" y2="36.96" width="0.8128" layer="1"/>
+<wire x1="21.53" y1="36.96" x2="21.53" y2="37.51" width="0.8128" layer="1"/>
 </signal>
 <signal name="AIN5">

Commit message: [ update ] notes
Other:
- board text added: "bbone_ct_cape"
Changed lines of the file:
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@@
 <wire x1="49.2" y1="49.52" x2="0" y2="49.52" width="0" layer="20"/>
 <wire x1="0" y1="49.52" x2="0" y2="0" width="0" layer="20"/>
-<text x="2.54" y="45.72" size="0.8128" layer="25">texane@gmail.com</text>
-<text x="2.54" y="46.99" size="0.8128" layer="25">v0000</text>
+<text x="2.54" y="44.45" size="0.8128" layer="25">texane@gmail.com</text>
+<text x="2.54" y="45.72" size="0.8128" layer="25">v0000</text>
+<text x="2.54" y="46.99" size="0.8128" layer="25">bbone_ct_cape</text>
 </plain>
 <attributes>

Commit message: [ update ] schematics revision
Other:
- board text added: "rev 91c018a3751a"
- board text removed: "v0000"
Changed lines of the file:
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@@
 <wire x1="0" y1="49.52" x2="0" y2="0" width="0" layer="20"/>
 <text x="2.54" y="44.45" size="0.8128" layer="25">texane@gmail.com</text>
-<text x="2.54" y="45.72" size="0.8128" layer="25">v0000</text>
+<text x="2.54" y="45.72" size="0.8128" layer="25">rev 91c018a3751a</text>
 <text x="2.54" y="46.99" size="0.8128" layer="25">bbone_ct_cape</text>
 </plain>
