File: sch/main.sch (EAGLE design)
At the start: 6 parts, among them X1 1503_02

Commit message: [ update ] sch
Other:
- note added: "BONE_SCH.pdf, AIN0, P9.39"
- note added: "BONE_SCH.pdf, GNDA_ADC, P9.34"
- note added: "BONE_SCH.pdf, VDD_ADC, P9.32"
Changed lines of the file:
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@@
 <layer number="95" name="Names" color="7" fill="1" visible="yes" active="yes"/>
 <layer number="96" name="Values" color="7" fill="1" visible="yes" active="yes"/>
-<layer number="97" name="Info" color="7" fill="1" visible="yes" active="yes"/>
+<layer number="97" name="Info" color="5" fill="1" visible="yes" active="yes"/>
 <layer number="98" name="Guide" color="6" fill="1" visible="yes" active="yes"/>
 </layers>
@@
 <text x="-17.78" y="68.58" size="1.778" layer="97">assumes Imax is 50A peak (35A RMS)</text>
 <text x="-17.78" y="66.04" size="1.778" layer="97">assumes SCT-013-000 sensor</text>
+<text x="25.4" y="93.98" size="1.778" layer="97">BONE_SCH.pdf, VDD_ADC, P9.32</text>
+<text x="30.48" y="50.8" size="1.778" layer="97">BONE_SCH.pdf, GNDA_ADC, P9.34</text>
+<text x="15.24" y="109.22" size="1.778" layer="97">BONE_SCH.pdf, AIN0, P9.39</text>
 </plain>
 <instances>

Commit message: [ update, add ] board
Parts:
- added JP1, JP10, JP11, JP2, JP3, JP4, JP5, JP6, JP7, JP8, JP9: M10LOCK, SparkFun:M10LOCK
- added P9: (no value), con-lstb:MA18-2
- added R3: 4.7K, rcl:R-EU_M1206
- added U1: (no value), SparkFun:TMP36TO-92-KIT
- R5: value 470 -> 1K
Connections:
- removed net ADC_0: R5.2
- removed net AVCC: R1.2
- new net AIN5: P9.36, R5.2
- new net GNDA_ADC: C2.2, P9.34, R2.1
- new net GPIO1_28: P9.12, R3.1, U1.VOUT
- new net VDD_3V3: P9.4, R3.2, U1.VCC
- new net VDD_5V: P9.6
- new net VDD_ADC: P9.32, R1.2
- net GND: now also P9.1, P9.2, U1.GND; no longer C2.2, R2.1
Other:
- note added: "actually a DS18B20+"
- note added: "free to use headers"

Commit message: [ update ] schematics
Other:
- note added: "texane@gmail.com"
- note added: "v0000"
- moved on the sheet: JP1, JP10, JP11, JP2, JP3, JP4, JP5, JP6, JP7, JP8, JP9
Changed lines of the file:
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@@
 <part name="JP10" library="SparkFun" deviceset="M10" device="LOCK"/>
 <part name="JP11" library="SparkFun" deviceset="M10" device="LOCK"/>
+<part name="FRAME1" library="frames" deviceset="A4L-LOC" device=""/>
 </parts>
 <sheets>
@@
 <text x="15.24" y="109.22" size="1.778" layer="97">BONE_SCH.pdf, AIN0, P9.39</text>
 <text x="15.24" y="121.92" size="1.778" layer="97">actually a DS18B20+</text>
-<text x="0" y="40.64" size="1.778" layer="97">free to use headers</text>
+<text x="132.08" y="137.16" size="1.778" layer="97">free to use headers</text>
+<text x="134.62" y="25.4" size="1.778" layer="94">texane@gmail.com</text>
+<text x="134.62" y="22.86" size="1.778" layer="94">v0000</text>
 </plain>
 <instances>
@@
 </instance>
 <instance part="R3" gate="G$1" x="38.1" y="134.62" rot="R90"/>
-<instance part="JP3" gate="G$1" x="0" y="27.94"/>
-<instance part="JP1" gate="G$1" x="12.7" y="27.94"/>
-<instance part="JP2" gate="G$1" x="25.4" y="27.94"/>
-<instance part="JP4" gate="G$1" x="38.1" y="27.94"/>
-<instance part="JP5" gate="G$1" x="0" y="-7.62"/>
-<instance part="JP6" gate="G$1" x="12.7" y="-7.62"/>
-<instance part="JP7" gate="G$1" x="25.4" y="-7.62"/>
-<instance part="JP8" gate="G$1" x="38.1" y="-7.62"/>
-<instance part="JP9" gate="G$1" x="50.8" y="-7.62"/>
+<instance part="JP3" gate="G$1" x="132.08" y="124.46"/>
+<instance part="JP1" gate="G$1" x="144.78" y="124.46"/>
+<instance part="JP2" gate="G$1" x="157.48" y="124.46"/>
+<instance part="JP4" gate="G$1" x="170.18" y="124.46"/>
+<instance part="JP5" gate="G$1" x="132.08" y="88.9"/>
+<instance part="JP6" gate="G$1" x="144.78" y="88.9"/>
+<instance part="JP7" gate="G$1" x="157.48" y="88.9"/>
+<instance part="JP8" gate="G$1" x="170.18" y="88.9"/>
+<instance part="JP9" gate="G$1" x="182.88" y="88.9"/>
 <instance part="P9" gate="G$1" x="88.9" y="99.06" rot="R180"/>
-<instance part="JP10" gate="G$1" x="50.8" y="27.94"/>
-<instance part="JP11" gate="G$1" x="63.5" y="27.94"/>
+<instance part="JP10" gate="G$1" x="182.88" y="124.46"/>
+<instance part="JP11" gate="G$1" x="195.58" y="124.46"/>
+<instance part="FRAME1" gate="G$1" x="-30.48" y="5.08" smashed="yes">
+<attribute name="DRAWING_NAME" x="186.69" y="20.32" size="2.54" layer="94" font="vector"/>
+<attribute name="LAST_DATE_TIME" x="186.69" y="15.24" size="2.286" layer="94" font="vector"/>
+<attribute name="SHEET" x="200.025" y="10.16" size="2.54" layer="94" font="vector"/>
+</instance>
 </instances>
 <busses>

Commit message: [ update ] notes
Other:
- note added: "https://github.com/texane/bbone_ct_cape"
Changed lines of the file:
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@@
 <text x="15.24" y="121.92" size="1.778" layer="97">actually a DS18B20+</text>
 <text x="132.08" y="137.16" size="1.778" layer="97">free to use headers</text>
-<text x="134.62" y="25.4" size="1.778" layer="94">texane@gmail.com</text>
+<text x="134.62" y="20.32" size="1.778" layer="94">texane@gmail.com</text>
 <text x="134.62" y="22.86" size="1.778" layer="94">v0000</text>
+<text x="134.62" y="25.4" size="1.778" layer="94">https://github.com/texane/bbone_ct_cape</text>
 </plain>
 <instances>

Commit message: [ update ] schematics revision
Other:
- note added: "rev 91c018a3751a"
- note removed: "v0000"
Changed lines of the file:
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@@
 <text x="132.08" y="137.16" size="1.778" layer="97">free to use headers</text>
 <text x="134.62" y="20.32" size="1.778" layer="94">texane@gmail.com</text>
-<text x="134.62" y="22.86" size="1.778" layer="94">v0000</text>
+<text x="134.62" y="22.86" size="1.778" layer="94">rev 91c018a3751a</text>
 <text x="134.62" y="25.4" size="1.778" layer="94">https://github.com/texane/bbone_ct_cape</text>
 </plain>
